File: output/pcbs/travis_num2024-route2.kicad_pcb (KiCad board)
At the start: 2 copper layers, 85.2 x 132.8 mm, 92 parts

Commit message: led fix
Routing:
- net LED_2: track 15.1 -> 16.2 mm
- net LED_1: track 15.1 -> 16.2 mm
- net LED_3: track 15.1 -> 15.7 mm
