File: output/pcbs/travis_num2024-route3.kicad_pcb (KiCad board)
At the start: 2 copper layers, 85.2 x 132.8 mm, 91 parts

Commit message: smd progress, labels added
Routing:
- net VCC: track 599.0 -> 619.3 mm, vias 6 -> 0
- net col0: track 131.7 -> 118.4 mm, vias 6 -> 9
- net col2: track 131.3 -> 121.5 mm, vias 6 -> 9
- net col1: track 101.1 -> 94.0 mm, vias 5 -> 7
- net LED_18: track 30.3 -> 26.1 mm
- net matrix_col1_row4: track 0.00 -> 2.58 mm
- net matrix_col0_row4: track 0.00 -> 2.58 mm
- net col3: track 167.0 -> 164.7 mm, vias 4 -> 5
- net LED_0: track 31.1 -> 29.4 mm
- net row4: track 63.4 -> 61.8 mm
- net LED_12: track 28.9 -> 29.4 mm
