File: output/pcbs/travis_num2024.kicad_pcb (KiCad board)
At the start: 2 copper layers, 85.2 x 132.8 mm, 92 parts

Commit message: working on plate
Parts:
- removed KC15, KC16, KC17: 104, Capacitor_THT:C_Disc_D4.7mm_W2.5mm_P5.00mm
- removed KD15, KD16, KD17: 1N4148, ScottoKeebs_Components:Diode_DO-35
- removed KSW15, KSW16, KSW17: Kailh MX Switch Sockets, travis:MX
- removed LED_11-row2-col3, LED_18-row0-col3, LED_20-row0-col0: SK6812mini-e, travis:led_SK6812mini-e
- moved KSW11 82.7 mm to (80.1, 200.0)
- moved KC11 82.7 mm to (77.6, 208.3)
- moved KD11 82.7 mm to (88.6, 192.0)
- moved KSW9 44.8 mm to (60.0, 159.9)
- moved KC9 44.8 mm to (57.5, 168.2)
- moved KD9 44.8 mm to (68.6, 151.9)
- moved KC7 41.3 mm to (37.5, 168.2)
- moved KSW7 41.3 mm to (40.0, 159.9)
- moved KD7 41.3 mm to (48.5, 151.9)
- moved KC12 40.1 mm to (77.6, 168.2)
- moved KSW12 40.1 mm to (80.1, 159.9)
- moved KSW10 40.1 mm to (60.0, 119.8)
- moved KSW13 40.1 mm to (80.1, 119.8)
- moved KSW8 40.1 mm to (40.0, 119.8)
- moved KC10 40.1 mm to (57.5, 128.1)
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Connections:
- KD10 pad 1: row2 -> row4
- KD10 pad 2: matrix_col1_row2 -> matrix_col1_row4
- KD11 pad 1: row4 -> row0
- KD11 pad 2: matrix_col1_row4 -> matrix_col2_row0
- KD12 pad 1: row0 -> row2
- KD12 pad 2: matrix_col2_row0 -> matrix_col2_row2
- KD13 pad 1: row2 -> row4
- KD13 pad 2: matrix_col2_row2 -> matrix_col2_row4
- KD14 pad 1: row4 -> row3
- KD14 pad 2: matrix_col2_row4 -> matrix_col3_row4
- KD7 pad 1: row0 -> row2
- KD7 pad 2: matrix_col0_row0 -> matrix_col0_row2
- KD8 pad 1: row2 -> row4
- KD8 pad 2: matrix_col0_row2 -> matrix_col0_row4
- KD9 pad 1: row4 -> row2
- KD9 pad 2: matrix_col0_row4 -> matrix_col1_row2
- KSW10 pad 2: matrix_col1_row2 -> matrix_col1_row4
- KSW11 pad 1: col1 -> col2
- KSW11 pad 2: matrix_col1_row4 -> matrix_col2_row0
- KSW12 pad 2: matrix_col2_row0 -> matrix_col2_row2
- KSW13 pad 2: matrix_col2_row2 -> matrix_col2_row4
- KSW14 pad 1: col2 -> col3
- KSW14 pad 2: matrix_col2_row4 -> matrix_col3_row4
- KSW7 pad 2: matrix_col0_row0 -> matrix_col0_row2
- KSW8 pad 2: matrix_col0_row2 -> matrix_col0_row4
- KSW9 pad 1: col0 -> col1
- KSW9 pad 2: matrix_col0_row4 -> matrix_col1_row2
Routing:
- net RAW: track 86.0 -> 67.0 mm, vias 11 -> 8
- net GND: track 68.0 -> 59.8 mm
- net matrix_col3_row0: track 5.79 -> 0.00 mm
- net matrix_col0_row0: track 5.79 -> 0.00 mm
- net matrix_col3_row2: track 5.79 -> 0.00 mm
Other:
- board text removed: "KC15"
- board text removed: "KC16"
- board text removed: "KC17"
- board text removed: "KD15"
- board text removed: "KD16"
- board text removed: "KD17"
- board text removed: "LED_11"
- board text removed: "LED_18"
- board text removed: "LED_20"
- board text removed: "matrix_col0_row0 col0 row0"
- board text removed: "matrix_col3_row0 col3 row0"
- board text removed: "matrix_col3_row2 col3 row2"

Commit message: new footprints for smd components
Parts:
- removed R1: 470R, Resistor_THT:R_Axial_DIN0207_L6.3mm_D2.5mm_P10.16mm_Horizontal
- added KC15: 104, Capacitor_THT:C_Disc_D4.7mm_W2.5mm_P5.00mm, B.Cu at (108.5, 192.5)
- added KC16: 104, Capacitor_THT:C_Disc_D4.7mm_W2.5mm_P5.00mm, B.Cu at (108.5, 152.4)
- added KC17: 104, Capacitor_THT:C_Disc_D4.7mm_W2.5mm_P5.00mm, B.Cu at (97.7, 128.1)
- added KD15: 1N4148, ScottoKeebs_Components:Diode_DO-35, B.Cu at (92.1, 181.4)
- added KD16: 1N4148, ScottoKeebs_Components:Diode_DO-35, B.Cu at (92.1, 141.3)
- added KD17: 1N4148, ScottoKeebs_Components:Diode_DO-35, B.Cu at (108.7, 111.8)
- added KSW15: Kailh MX Switch Sockets, travis:MX, F.Cu at (100.2, 190.0)
- added KSW16: Kailh MX Switch Sockets, travis:MX, F.Cu at (100.2, 149.9)
- added KSW17: Kailh MX Switch Sockets, travis:MX, F.Cu at (100.2, 119.8)
- added LED_11-row2-col3: SK6812mini-e, travis:led_SK6812mini-e, B.Cu at (105.1, 149.9)
- added LED_18-row0-col3: SK6812mini-e, travis:led_SK6812mini-e, B.Cu at (105.1, 190.0)
- added LED_20-row0-col0: SK6812mini-e, travis:led_SK6812mini-e, B.Cu at (50.0, 205.0)
- C1: value 6.3V 1000uF -> 470uF 10V; footprint Capacitor_THT:C_Radial_D6.3mm_H11.0mm_P2.50mm -> CP_Elec_6.3x7.7; moved to F.Cu
- C2, C3, C4, C5: value 104 -> C_1206_3216Metric; footprint Capacitor_THT:C_Disc_D4.7mm_W2.5mm_P5.00mm -> C_1206_3216Metric
- D1: value 1N4148 -> (none); footprint ScottoKeebs_Components:Diode_DO-35 -> ceoloide:diode_tht_sod123
- LOGO1: footprint ceoloide:ergogen_logo -> ceoloide:utility_ergogen_logo
- moved KSW11 82.7 mm to (60.0, 119.8)
- moved KC11 82.7 mm to (57.5, 128.1)
- moved KD11 82.7 mm to (68.6, 111.8)
- moved KSW9 44.8 mm to (40.0, 119.8)
- moved KC9 44.8 mm to (37.5, 128.1)
- moved KD9 44.8 mm to (48.5, 111.8)
- moved KC7 41.3 mm to (47.5, 208.3)
- moved KSW7 41.3 mm to (50.0, 200.0)
- moved KD7 41.3 mm to (58.5, 192.0)
- moved KC12 40.1 mm to (77.6, 208.3)
- moved KSW12 40.1 mm to (80.1, 200.0)
- moved KSW10 40.1 mm to (60.0, 159.9)
- moved KSW13 40.1 mm to (80.1, 159.9)
- moved KSW8 40.1 mm to (40.0, 159.9)
- moved KC10 40.1 mm to (57.5, 168.2)
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Connections:
- C1 pad 1: RAW -> VCC
- C2 pad 1: RAW -> VCC
- C3 pad 1: RAW -> VCC
- C4 pad 1: RAW -> VCC
- C5 pad 1: RAW -> VCC
- KD10 pad 1: row4 -> row2
- KD10 pad 2: matrix_col1_row4 -> matrix_col1_row2
- KD11 pad 1: row0 -> row4
- KD11 pad 2: matrix_col2_row0 -> matrix_col1_row4
- KD12 pad 1: row2 -> row0
- KD12 pad 2: matrix_col2_row2 -> matrix_col2_row0
- KD13 pad 1: row4 -> row2
- KD13 pad 2: matrix_col2_row4 -> matrix_col2_row2
- KD14 pad 1: row3 -> row4
- KD14 pad 2: matrix_col3_row4 -> matrix_col2_row4
- KD7 pad 1: row2 -> row0
- KD7 pad 2: matrix_col0_row2 -> matrix_col0_row0
- KD8 pad 1: row4 -> row2
- KD8 pad 2: matrix_col0_row4 -> matrix_col0_row2
- KD9 pad 1: row2 -> row4
- KD9 pad 2: matrix_col1_row2 -> matrix_col0_row4
- KSW10 pad 2: matrix_col1_row4 -> matrix_col1_row2
- KSW11 pad 1: col2 -> col1
- KSW11 pad 2: matrix_col2_row0 -> matrix_col1_row4
- KSW12 pad 2: matrix_col2_row2 -> matrix_col2_row0
- KSW13 pad 2: matrix_col2_row4 -> matrix_col2_row2
- KSW14 pad 1: col3 -> col2
- KSW14 pad 2: matrix_col3_row4 -> matrix_col2_row4
- KSW7 pad 2: matrix_col0_row2 -> matrix_col0_row0
- KSW8 pad 2: matrix_col0_row4 -> matrix_col0_row2
- KSW9 pad 1: col1 -> col0
- KSW9 pad 2: matrix_col1_row2 -> matrix_col0_row4
- LED1 pad 1: RAW -> VCC
- LED2 pad 1: RAW -> VCC
- LED3 pad 1: RAW -> VCC
- LED4 pad 1: RAW -> VCC
- MCU1 pad 12: LED -> LED0
Routing:
- net RAW: track 67.0 -> 86.0 mm, vias 8 -> 11
- net GND: track 59.8 -> 68.0 mm
- net matrix_col3_row0: track 0.00 -> 5.79 mm
- net matrix_col0_row0: track 0.00 -> 5.79 mm
- net matrix_col3_row2: track 0.00 -> 5.79 mm
Other:
- net class Default removed
- board text added: "2024.05.10"
- board text added: "KC15"
- board text added: "KC16"
- board text added: "KC17"
- board text added: "KD15"
- board text added: "KD16"
- board text added: "KD17"
- board text added: "LED_11"
- board text added: "LED_18"
- board text added: "LED_20"
- board text added: "github.com/dieseltravis/travis-ergonum"
- board text added: "matrix_col0_row0 col0 row0"
- board text added: "matrix_col3_row0 col3 row0"
- board text added: "matrix_col3_row2 col3 row2"
- board text removed: "2024.04.13"

Commit message: smd progress
Parts:
- removed KC12, KC13, KC14, KC15, KC16, KC17: 104, Capacitor_THT:C_Disc_D4.7mm_W2.5mm_P5.00mm
- removed KD12, KD13, KD14, KD15, KD16, KD17: 1N4148, ScottoKeebs_Components:Diode_DO-35
- removed KSW12, KSW13, KSW14, KSW15, KSW16, KSW17: Kailh MX Switch Sockets, travis:MX
- removed LED_10-row3-col2, LED_15-row1-col0, LED_16-row1-col1, LED_17-row1-col2, LED_8-row3-col0, LED_9-row3-col1: SK6812mini-e, travis:led_SK6812mini-e
- added C10: C_1206_3216Metric, C_1206_3216Metric, B.Cu at (77.6, 188.2)
- added C11: C_1206_3216Metric, C_1206_3216Metric, B.Cu at (77.6, 148.1)
- added C6: C_1206_3216Metric, C_1206_3216Metric, B.Cu at (37.5, 188.2)
- added C7: C_1206_3216Metric, C_1206_3216Metric, B.Cu at (37.5, 148.1)
- added C8: C_1206_3216Metric, C_1206_3216Metric, B.Cu at (57.5, 188.2)
- added C9: C_1206_3216Metric, C_1206_3216Metric, B.Cu at (57.5, 148.1)
- added D2: D_1206_3216Metric, D_1206_3216Metric, B.Cu at (48.5, 131.8)
- added D3: D_1206_3216Metric, D_1206_3216Metric, B.Cu at (68.6, 171.9)
- added D4: D_1206_3216Metric, D_1206_3216Metric, B.Cu at (68.6, 131.8)
- added D5: D_1206_3216Metric, D_1206_3216Metric, B.Cu at (88.6, 171.9)
- added D6: D_1206_3216Metric, D_1206_3216Metric, B.Cu at (88.6, 131.8)
- added D7: D_1206_3216Metric, D_1206_3216Metric, B.Cu at (92.1, 94.7)
- added LED10: SK6812mini-e, travis:led_SK6812mini-e (per-key, single-side), B.Cu at (80.1, 144.8)
- added LED5: SK6812mini-e, travis:led_SK6812mini-e (per-key, single-side), B.Cu at (40.0, 184.9)
- added LED6: SK6812mini-e, travis:led_SK6812mini-e (per-key, single-side), B.Cu at (40.0, 144.8)
- added LED7: SK6812mini-e, travis:led_SK6812mini-e (per-key, single-side), B.Cu at (60.0, 184.9)
- added LED8: SK6812mini-e, travis:led_SK6812mini-e (per-key, single-side), B.Cu at (60.0, 144.8)
- added LED9: SK6812mini-e, travis:led_SK6812mini-e (per-key, single-side), B.Cu at (80.1, 184.9)
- added S1: Kailh MX Switch Sockets, travis:MX, F.Cu at (40.0, 179.9)
- added S2: Kailh MX Switch Sockets, travis:MX, F.Cu at (40.0, 139.8)
- added S3: Kailh MX Switch Sockets, travis:MX, F.Cu at (60.0, 179.9)
- added S4: Kailh MX Switch Sockets, travis:MX, F.Cu at (60.0, 139.8)
- added S5: Kailh MX Switch Sockets, travis:MX, F.Cu at (80.1, 179.9)
- added S6: Kailh MX Switch Sockets, travis:MX, F.Cu at (80.1, 139.8)
- D1: value (none) -> D_1206_3216Metric; footprint ceoloide:diode_tht_sod123 -> D_1206_3216Metric
- moved KC9 95.8 mm to (108.5, 192.5), turned to 90 degrees
- moved KSW9 92.4 mm to (100.2, 190.0), turned to 90 degrees
- moved D1 88.6 mm to (48.5, 171.9)
- moved KD9 82.2 mm to (92.1, 181.4), turned to 360 degrees
- moved KC3 65.2 mm to (37.5, 128.1), turned to 0 degrees
- moved KC5 65.2 mm to (57.5, 128.1), turned to 0 degrees
- moved KD3 63.4 mm to (48.5, 111.8)
- moved KD5 63.4 mm to (68.6, 111.8)
- moved KSW3 63.4 mm to (40.0, 119.8)
- moved KSW5 63.4 mm to (60.0, 119.8)
- moved KC6 60.4 mm to (77.6, 208.3), turned to 0 degrees
- moved KSW6 60.2 mm to (80.1, 200.0)
- moved KD6 60.2 mm to (88.6, 192.0)
- moved KSW8 56.7 mm to (80.1, 119.8)
- moved KC8 56.7 mm to (77.6, 128.1)
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Connections:
- D1 pad 1: row4 -> row1
- D1 pad 2: enc_to -> matrix_col0_row1
- KD1 pad 1: row1 -> row0
- KD1 pad 2: matrix_col0_row1 -> matrix_col0_row0
- KD10 pad 2: matrix_col1_row2 -> matrix_col3_row2
- KD11 pad 1: row4 -> row3
- KD11 pad 2: matrix_col1_row4 -> matrix_col3_row4
- KD2 pad 1: row3 -> row2
- KD2 pad 2: matrix_col0_row3 -> matrix_col0_row2
- KD3 pad 1: row1 -> row4
- KD3 pad 2: matrix_col1_row1 -> matrix_col0_row4
- KD4 pad 1: row3 -> row2
- KD4 pad 2: matrix_col1_row3 -> matrix_col1_row2
- KD5 pad 1: row1 -> row4
- KD5 pad 2: matrix_col2_row1 -> matrix_col1_row4
- KD6 pad 1: row3 -> row0
- KD6 pad 2: matrix_col2_row3 -> matrix_col2_row0
- KD7 pad 1: row0 -> row2
- KD7 pad 2: matrix_col0_row0 -> matrix_col2_row2
- KD8 pad 1: row2 -> row4
- KD8 pad 2: matrix_col0_row2 -> matrix_col2_row4
- KD9 pad 1: row4 -> row0
- KD9 pad 2: matrix_col0_row4 -> matrix_col3_row0
- KSW1 pad 2: matrix_col0_row1 -> matrix_col0_row0
- KSW10 pad 1: col1 -> col3
- KSW10 pad 2: matrix_col1_row2 -> matrix_col3_row2
- KSW11 pad 1: col1 -> col3
- KSW11 pad 2: matrix_col1_row4 -> matrix_col3_row4
- KSW2 pad 2: matrix_col0_row3 -> matrix_col0_row2
- KSW3 pad 1: col1 -> col0
- KSW3 pad 2: matrix_col1_row1 -> matrix_col0_row4
- KSW4 pad 2: matrix_col1_row3 -> matrix_col1_row2
- KSW5 pad 1: col2 -> col1
- KSW5 pad 2: matrix_col2_row1 -> matrix_col1_row4
- KSW6 pad 2: matrix_col2_row3 -> matrix_col2_row0
- KSW7 pad 1: col0 -> col2
- KSW7 pad 2: matrix_col0_row0 -> matrix_col2_row2
- KSW8 pad 1: col0 -> col2
- KSW8 pad 2: matrix_col0_row2 -> matrix_col2_row4
- KSW9 pad 1: col0 -> col3
- KSW9 pad 2: matrix_col0_row4 -> matrix_col3_row0
Routing:
- net GND: track 68.0 -> 30.0 mm, vias 6 -> 0
- net RAW: track 86.0 -> 69.7 mm
- net matrix_col2_row3: track 5.79 -> 0.00 mm
- net matrix_col2_row1: track 5.79 -> 0.00 mm
- net matrix_col1_row3: track 5.79 -> 0.00 mm
- net matrix_col1_row1: track 5.79 -> 0.00 mm
- net matrix_col0_row3: track 5.79 -> 0.00 mm
- net matrix_col0_row1: track 5.79 -> 0.00 mm
Other:
- board text removed: "KC12"
- board text removed: "KC13"
- board text removed: "KC14"
- board text removed: "KC15"
- board text removed: "KC16"
- board text removed: "KC17"
- board text removed: "KD12"
- board text removed: "KD13"
- board text removed: "KD14"
- board text removed: "KD15"
- board text removed: "KD16"
- board text removed: "KD17"
- board text removed: "matrix_col0_row1 col0 row1"
- board text removed: "matrix_col0_row3 col0 row3"
- board text removed: "matrix_col1_row1 col1 row1"
- board text removed: "matrix_col1_row3 col1 row3"
- board text removed: "matrix_col2_row1 col2 row1"
- board text removed: "matrix_col2_row3 col2 row3"

Commit message: smd progress
Parts:
- moved D7 8.23 mm to (94.4, 102.6), turned to 0 degrees
- moved C6 6.91 mm to (44.4, 187.3)
- moved C7 6.91 mm to (44.4, 147.2)
- moved C10 6.91 mm to (84.4, 187.3)
- moved C11 6.91 mm to (84.4, 147.2)
- moved C8 6.91 mm to (64.4, 187.3)
- moved C9 6.91 mm to (64.4, 147.2)
- moved D1 1.92 mm to (48.3, 173.8)
- moved D2 1.92 mm to (48.3, 133.7)
- moved D3 1.92 mm to (68.3, 173.8)
- moved D4 1.92 mm to (68.3, 133.7)
- moved D5 1.92 mm to (88.4, 173.8)
- moved D6 1.92 mm to (88.4, 133.7)

Commit message: smd progress
Parts:
- removed KC1, KC10, KC11, KC2, KC3, KC4, KC5, KC6, KC7, KC8, KC9: 104, Capacitor_THT:C_Disc_D4.7mm_W2.5mm_P5.00mm
- removed KD1, KD10, KD11, KD2, KD3, KD4, KD5, KD6, KD7, KD8, KD9: 1N4148, ScottoKeebs_Components:Diode_DO-35
- removed KSW1, KSW10, KSW11, KSW2, KSW3, KSW4, KSW5, KSW6, KSW7, KSW8, KSW9: Kailh MX Switch Sockets, travis:MX
- removed LED_11-row2-col3, LED_12-row2-col2, LED_13-row2-col1, LED_14-row2-col0, LED_18-row0-col3, LED_19-row0-col2, LED_20-row0-col0, LED_4-row3-col3, LED_5-row4-col2, LED_6-row4-col1, LED_7-row4-col0: SK6812mini-e, travis:led_SK6812mini-e
- added C12: C_1206_3216Metric, C_1206_3216Metric, B.Cu at (45.7, 202.6)
- added C13: C_1206_3216Metric, C_1206_3216Metric, B.Cu at (35.6, 162.5)
- added C14: C_1206_3216Metric, C_1206_3216Metric, B.Cu at (35.6, 122.4)
- added C15: C_1206_3216Metric, C_1206_3216Metric, B.Cu at (55.7, 162.5)
- added C16: C_1206_3216Metric, C_1206_3216Metric, B.Cu at (55.7, 122.4)
- added C17: C_1206_3216Metric, C_1206_3216Metric, B.Cu at (75.8, 202.6)
- added C18: C_1206_3216Metric, C_1206_3216Metric, B.Cu at (75.8, 162.5)
- added C19: C_1206_3216Metric, C_1206_3216Metric, B.Cu at (75.8, 122.4)
- added C20: C_1206_3216Metric, C_1206_3216Metric, B.Cu at (102.7, 194.3)
- added C21: C_1206_3216Metric, C_1206_3216Metric, B.Cu at (102.7, 154.2)
- added C22: C_1206_3216Metric, C_1206_3216Metric, B.Cu at (95.8, 122.4)
- added D10: D_1206_3216Metric, D_1206_3216Metric, B.Cu at (88.4, 193.9)
- added D11: D_1206_3216Metric, D_1206_3216Metric, B.Cu at (88.4, 173.8)
- added D12: D_1206_3216Metric, D_1206_3216Metric, B.Cu at (88.4, 153.8)
- added D13: D_1206_3216Metric, D_1206_3216Metric, B.Cu at (88.4, 133.7)
- added D14: D_1206_3216Metric, D_1206_3216Metric, B.Cu at (88.4, 113.7)
- added D15: D_1206_3216Metric, D_1206_3216Metric, B.Cu at (94.0, 181.7)
- added D16: D_1206_3216Metric, D_1206_3216Metric, B.Cu at (94.0, 141.6)
- added D17: D_1206_3216Metric, D_1206_3216Metric, B.Cu at (108.4, 113.7)
- added D18: D_1206_3216Metric, D_1206_3216Metric, B.Cu at (94.4, 102.6)
- added D8: D_1206_3216Metric, D_1206_3216Metric, B.Cu at (68.3, 133.7)
- added D9: D_1206_3216Metric, D_1206_3216Metric, B.Cu at (68.3, 113.7)
- added LED11: SK6812mini-e, travis:led_SK6812mini-e (per-key, single-side), B.Cu at (50.0, 205.0)
- added LED12: SK6812mini-e, travis:led_SK6812mini-e (per-key, single-side), B.Cu at (40.0, 164.9)
- added LED13: SK6812mini-e, travis:led_SK6812mini-e (per-key, single-side), B.Cu at (40.0, 124.8)
- added LED14: SK6812mini-e, travis:led_SK6812mini-e (per-key, single-side), B.Cu at (60.0, 164.9)
- added LED15: SK6812mini-e, travis:led_SK6812mini-e (per-key, single-side), B.Cu at (60.0, 124.8)
- added LED16: SK6812mini-e, travis:led_SK6812mini-e (per-key, single-side), B.Cu at (80.1, 205.0)
- added LED17: SK6812mini-e, travis:led_SK6812mini-e (per-key, single-side), B.Cu at (80.1, 164.9)
- added LED18: SK6812mini-e, travis:led_SK6812mini-e (per-key, single-side), B.Cu at (80.1, 124.8)
- added LED19: SK6812mini-e, travis:led_SK6812mini-e (per-key, single-side), B.Cu at (105.1, 190.0)
- added LED20: SK6812mini-e, travis:led_SK6812mini-e (per-key, single-side), B.Cu at (105.1, 149.9)
- added LED21: SK6812mini-e, travis:led_SK6812mini-e (per-key, single-side), B.Cu at (100.2, 124.8)
- added S10: Kailh MX Switch Sockets, travis:MX, F.Cu at (80.1, 200.0)
- added S11: Kailh MX Switch Sockets, travis:MX, F.Cu at (80.1, 179.9)
- added S12: Kailh MX Switch Sockets, travis:MX, F.Cu at (80.1, 159.9)
- added S13: Kailh MX Switch Sockets, travis:MX, F.Cu at (80.1, 139.8)
- added S14: Kailh MX Switch Sockets, travis:MX, F.Cu at (80.1, 119.8)
- added S15: Kailh MX Switch Sockets, travis:MX, F.Cu at (100.2, 190.0)
- added S16: Kailh MX Switch Sockets, travis:MX, F.Cu at (100.2, 149.9)
- added S17: Kailh MX Switch Sockets, travis:MX, F.Cu at (100.2, 119.8)
- added S7: Kailh MX Switch Sockets, travis:MX, F.Cu at (60.0, 159.9)
- added S8: Kailh MX Switch Sockets, travis:MX, F.Cu at (60.0, 139.8)
- added S9: Kailh MX Switch Sockets, travis:MX, F.Cu at (60.0, 119.8)
- moved D5 72.3 mm to (48.3, 113.7)
- moved S5 72.3 mm to (40.0, 119.8)
- moved D7 57.4 mm to (68.3, 153.8), turned to 270 degrees
- moved D6 44.8 mm to (68.3, 173.8)
- moved S6 44.8 mm to (60.0, 179.9)
- moved D2 40.1 mm to (48.3, 173.8)
- moved S2 40.1 mm to (40.0, 179.9)
- moved D3 28.4 mm to (48.3, 153.8)
- moved S3 28.4 mm to (40.0, 159.9)
- moved D1 22.4 mm to (58.3, 193.9)
- moved S1 22.4 mm to (50.0, 200.0)
- moved D4 20.1 mm to (48.3, 133.7)
- moved S4 20.0 mm to (40.0, 139.8)
Connections:
- D1 pad 1: row1 -> row0
- D1 pad 2: matrix_col0_row1 -> matrix_col0_row0
- D2 pad 1: row3 -> row1
- D2 pad 2: matrix_col0_row3 -> matrix_col0_row1
- D3 pad 1: row1 -> row2
- D3 pad 2: matrix_col1_row1 -> matrix_col0_row2
- D4 pad 2: matrix_col1_row3 -> matrix_col0_row3
- D5 pad 1: row1 -> row4
- D5 pad 2: matrix_col2_row1 -> matrix_col0_row4
- D6 pad 1: row3 -> row1
- D6 pad 2: matrix_col2_row3 -> matrix_col1_row1
- D7 pad 1: row4 -> row2
- D7 pad 2: enc_to -> matrix_col1_row2
- MCU1 pad 12: LED0 -> LED_0
- S1 pad 2: matrix_col0_row1 -> matrix_col0_row0
- S2 pad 2: matrix_col0_row3 -> matrix_col0_row1
- S3 pad 1: col1 -> col0
- S3 pad 2: matrix_col1_row1 -> matrix_col0_row2
- S4 pad 1: col1 -> col0
- S4 pad 2: matrix_col1_row3 -> matrix_col0_row3
- S5 pad 1: col2 -> col0
- S5 pad 2: matrix_col2_row1 -> matrix_col0_row4
- S6 pad 1: col2 -> col1
- S6 pad 2: matrix_col2_row3 -> matrix_col1_row1
Routing:
- net RAW: track 69.7 -> 0.00 mm, vias 11 -> 0
- net GND: track 30.0 -> 0.00 mm
- net matrix_col3_row0: track 5.79 -> 0.00 mm
- net matrix_col2_row2: track 5.79 -> 0.00 mm
- net matrix_col2_row0: track 5.79 -> 0.00 mm
- net matrix_col1_row2: track 5.79 -> 0.00 mm
- net matrix_col0_row2: track 5.79 -> 0.00 mm
- net matrix_col0_row0: track 5.79 -> 0.00 mm
- net matrix_col3_row2: track 5.79 -> 0.00 mm
- net matrix_col2_row4: track 5.79 -> 0.00 mm
- net matrix_col1_row4: track 5.79 -> 0.00 mm
- net matrix_col0_row4: track 5.79 -> 0.00 mm
- net matrix_col3_row4: track 5.79 -> 0.00 mm
Other:
- board text removed: "KC1"
- board text removed: "KC10"
- board text removed: "KC11"
- board text removed: "KC2"
- board text removed: "KC3"
- board text removed: "KC4"
- board text removed: "KC5"
- board text removed: "KC6"
- board text removed: "KC7"
- board text removed: "KC8"
- board text removed: "KC9"
- board text removed: "KD1"
- board text removed: "KD10"
- board text removed: "KD11"
- board text removed: "KD2"
- board text removed: "KD3"
- board text removed: "KD4"
- board text removed: "KD5"
- board text removed: "KD6"
- board text removed: "KD7"
- board text removed: "KD8"
- board text removed: "KD9"
- board text removed: "matrix_col0_row0 col0 row0"
- board text removed: "matrix_col0_row2 col0 row2"
- board text removed: "matrix_col0_row4 col0 row4"
- board text removed: "matrix_col1_row2 col1 row2"
- board text removed: "matrix_col1_row4 col1 row4"
- board text removed: "matrix_col2_row0 col2 row0"
- board text removed: "matrix_col2_row2 col2 row2"
- board text removed: "matrix_col2_row4 col2 row4"
- board text removed: "matrix_col3_row0 col3 row0"
- board text removed: "matrix_col3_row2 col3 row2"
- board text removed: "matrix_col3_row4 col3 row3"

Commit message: smd progress, labels added
Parts:
- moved D1 0.15 mm to (58.5, 193.9)
- moved D15 0.15 mm to (94.0, 181.5)
- moved D16 0.15 mm to (94.0, 141.4)
- moved D2 0.15 mm to (48.4, 173.8)
- moved D3 0.15 mm to (48.4, 153.8)
- moved D4 0.15 mm to (48.4, 133.7)
- moved D5 0.15 mm to (48.4, 113.7)
- moved D10 0.15 mm to (88.5, 193.9)
- moved D11 0.15 mm to (88.5, 173.8)
- moved D12 0.15 mm to (88.5, 153.8)
- moved D13 0.15 mm to (88.5, 133.7)
- moved D14 0.15 mm to (88.5, 113.7)
- moved D17 0.15 mm to (108.6, 113.7)
- moved D6 0.15 mm to (68.5, 173.8)
- moved D7 0.15 mm to (68.5, 153.8)
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Other:
- board text added: "2024.05.15"
- board text added: "col0 row0"
- board text added: "col0 row1"
- board text added: "col0 row2"
- board text added: "col0 row3"
- board text added: "col0 row4"
- board text added: "col1 row1"
- board text added: "col1 row2"
- board text added: "col1 row3"
- board text added: "col1 row4"
- board text added: "col2 row0"
- board text added: "col2 row1"
- board text added: "col2 row2"
- board text added: "col2 row3"
- board text added: "col2 row4"
- board text added: "col3 row0"
- board text added: "col3 row2"
- board text added: "col3 row3"
- board text added: "github.com/dieseltravis/travis-ergogen-numpad"
- board text removed: "2024.05.10"
- board text removed: "github.com/dieseltravis/travis-ergonum"

Commit message: routed
Routing:
- net VCC: track 0.00 -> 620.9 mm
- net col3: track 0.00 -> 163.0 mm, vias 0 -> 5
- net row0: track 0.00 -> 142.6 mm, vias 0 -> 1
- net col2: track 0.00 -> 124.3 mm, vias 0 -> 8
- net col0: track 0.00 -> 119.3 mm, vias 0 -> 9
- net row1: track 0.00 -> 114.3 mm, vias 0 -> 1
- net row3: track 0.00 -> 108.7 mm, vias 0 -> 1
- net row2: track 0.00 -> 105.9 mm, vias 0 -> 1
- net col1: track 0.00 -> 94.9 mm, vias 0 -> 7
- net row4: track 0.00 -> 63.5 mm, vias 0 -> 3
- net encA: track 0.00 -> 47.2 mm
- net encC: track 0.00 -> 41.8 mm
- net LED_0: track 0.00 -> 30.4 mm
- net LED_18: track 0.00 -> 30.3 mm
- net LED_11: track 0.00 -> 30.3 mm
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Other:
- board text added: "S1"
- board text added: "S10"
- board text added: "S11"
- board text added: "S12"
- board text added: "S13"
- board text added: "S14"
- board text added: "S15"
- board text added: "S16"
- board text added: "S17"
- board text added: "S2"
- board text added: "S3"
- board text added: "S4"
- board text added: "S5"
- board text added: "S6"
- board text added: "S7"
- board text added: "S8"
- board text added: "S9"

Commit message: routed
Routing:
- net VCC: track 620.9 -> 0.00 mm
- net col3: track 163.0 -> 0.00 mm, vias 5 -> 0
- net row0: track 142.6 -> 0.00 mm, vias 1 -> 0
- net col2: track 124.3 -> 0.00 mm, vias 8 -> 0
- net col0: track 119.3 -> 0.00 mm, vias 9 -> 0
- net row1: track 114.3 -> 0.00 mm, vias 1 -> 0
- net row3: track 108.7 -> 0.00 mm, vias 1 -> 0
- net row2: track 105.9 -> 0.00 mm, vias 1 -> 0
- net col1: track 94.9 -> 0.00 mm, vias 7 -> 0
- net row4: track 63.5 -> 0.00 mm, vias 3 -> 0
- net encA: track 47.2 -> 0.00 mm
- net encC: track 41.8 -> 0.00 mm
- net LED_0: track 30.4 -> 0.00 mm
- net LED_18: track 30.3 -> 0.00 mm
- net LED_11: track 30.3 -> 0.00 mm
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