File: output/pcbs/travis_num2024-routed2.kicad_pcb (KiCad board)
At the start: 2 copper layers, 85.2 x 137.8 mm, 91 parts

Commit message: added qmk led layout & recompiled for ce
Parts:
- renumbered LED1 to LED_0, LED2 to LED_1, LED10 to LED_10, LED20 to LED_11, LED17 to LED_12, LED14 to LED_13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
